File: manufacturing/Reader_Module/Antenna.kicad_sch (KiCad schematic)
At the start: 0 parts

Commit message: added Matching NW to Schematic
Parts:
- added AE1: Antenna_Loop, RF_Antenna:Custom_RFID_1, symbol Device:Antenna_Loop
- added C25: 47p, Capacitor_SMD:C_0402_1005Metric, symbol Device:C
- added C26: 27p, Capacitor_SMD:C_0402_1005Metric, symbol Device:C
- added C27: 68p, Capacitor_SMD:C_0402_1005Metric, symbol Device:C
- added R10: 680R, Resistor_SMD:R_0402_1005Metric, symbol Device:R
Connections:
- net ANT_IN: now also C27.1
- new net Antenna: AE1.1, C25.1, C26.1, C27.2, R10.1
- new net GND: AE1.2, C25.2, C26.2, R10.2
Other:
- note added: "TI Application Note: SLOA241C"
- note added: "Website: https://eds.st.com/antenna/#/"
- company: (none) -> s-grundner
- title: (none) -> RFID-Gwent: Reader Module Antenna

Commit message: upd board
Parts:
- C25: LCSC Part # (none) -> C1567
- C26: LCSC Part # (none) -> C1557
- C27: LCSC Part # (none) -> C14441
- R10: LCSC Part # (none) -> C25130
Changed lines of the file:
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@@
+      (effects (font (size 1.27 1.27)) hide)
+    )
+    (property "LCSC Part #" "C1557" (at 95.25 96.52 0)
       (effects (font (size 1.27 1.27)) hide)
     )
@@
       (effects (font (size 1.27 1.27)) hide)
     )
+    (property "LCSC Part #" "C1567" (at 105.41 96.52 0)
+      (effects (font (size 1.27 1.27)) hide)
+    )
     (pin "1")
     (pin "2")
@@
     )
     (property "Datasheet" "~" (at 80.01 91.44 0)
+      (effects (font (size 1.27 1.27)) hide)
+    )
+    (property "LCSC Part #" "C14441" (at 80.01 91.44 0)
       (effects (font (size 1.27 1.27)) hide)
     )
@@
       (effects (font (size 1.27 1.27)) hide)
     )
+    (property "LCSC Part #" "C25130" (at 85.09 96.52 0)
+      (effects (font (size 1.27 1.27)) hide)
+    )
