File: manufacturing/Reader_Module/CAN.kicad_sch (KiCad schematic)
At the start: 14 parts, among them J2 Conn_01x04_Pin, U3 SN65HVD230, U4 USBLC6-2

Commit message: added Matching NW to Schematic
Parts:
- added C28, C29: 2u2, Capacitor_SMD:C_0402_1005Metric, symbol Device:C_Small
- added FB1: 100 @ 100MHz, Inductor_SMD:L_0805_2012Metric, symbol Device:FerriteBead_Small
- J2: footprint Connector_Molex:Molex_Micro-Latch_53253-0470_1x04_P2.00mm_Vertical -> Connector_Molex:Molex_Micro-Latch_53254-0470_1x04_P2.00mm_Horizontal
- R1: footprint Resistor_SMD:R_0805_2012Metric -> Resistor_SMD:R_0402_1005Metric
Connections:
- net +5V: now also C28.1, FB1.1; no longer J2.1 (Pin_1), U4.5
- net CAN_CON+: now also J2.3 (Pin_3); no longer J2.2 (Pin_2)
- net CAN_CON-: now also J2.2 (Pin_2); no longer J2.3 (Pin_3)
- net GND: now also J2.1 (Pin_1), C28.2, C29.2; no longer J2.4 (Pin_4)
- new net CONN_5V: C29.1, FB1.2, J2.4 (Pin_4), U4.5

Commit message: upd board
Parts:
- C28, C29: LCSC Part # (none) -> C2997286
- C6: LCSC Part # C1525 -> C2997286
- R1: value 47R -> 56R; LCSC Part # C25118 -> C25127
- R1: LCSC Part # C17757 -> C25127
Changed lines of the file:
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@@
       (effects (font (size 1.27 1.27)))
     )
-    (property "Value" "47R" (at 77.47 64.77 90)
+    (property "Value" "56R" (at 77.47 64.77 90)
       (effects (font (size 1.27 1.27)) (justify top))
     )
@@
       (effects (font (size 1.27 1.27)) hide)
     )
-    (property "LCSC Part #" "C25118" (at 77.47 66.04 0)
+    (property "LCSC Part #" "C25127" (at 77.47 66.04 0)
       (effects (font (size 1.27 1.27)) hide)
     )
@@
     )
     (property "Datasheet" "~" (at 147.32 58.42 0)
+      (effects (font (size 1.27 1.27)) hide)
+    )
+    (property "LCSC Part #" "C2997286" (at 147.32 58.42 0)
       (effects (font (size 1.27 1.27)) hide)
     )
@@
       (effects (font (size 1.27 1.27)) hide)
     )
-    (property "LCSC Part #" "C17757" (at 125.73 66.04 0)
+    (property "LCSC Part #" "C25127" (at 125.73 66.04 0)
       (effects (font (size 1.27 1.27)) hide)
     )
@@
       (effects (font (size 1.27 1.27)) hide)
     )
-    (property "LCSC Part #" "C1525" (at 36.83 69.85 0)
+    (property "LCSC Part #" "C2997286" (at 36.83 69.85 0)
       (effects (font (size 1.27 1.27)) hide)
     )
@@
       (effects (font (size 1.27 1.27)) hide)
     )
-    (property "LCSC Part #" "C17757" (at 125.73 73.66 0)
+    (property "LCSC Part #" "C25127" (at 125.73 73.66 0)
       (effects (font (size 1.27 1.27)) hide)
     )
@@
       (effects (font (size 1.27 1.27)) hide)
     )
+    (property "LCSC Part #" "C2997286" (at 160.02 58.42 0)
+      (effects (font (size 1.27 1.27)) hide)
+    )
     (pin "1")
     (pin "2")
@@
       (effects (font (size 1.27 1.27)))
     )
-    (property "Value" "47R" (at 77.47 72.39 90)
+    (property "Value" "56R" (at 77.47 72.39 90)
       (effects (font (size 1.27 1.27)) (justify top))
     )
@@
       (effects (font (size 1.27 1.27)) hide)
     )
-    (property "LCSC Part #" "C25118" (at 77.47 73.66 0)
-      (effects (font (size 1.27 1.27)) hide)
-    )
+    (property "LCSC Part #" "C25127" (at 77.47 73.66 0)
+      (effects (font (size 1.27 1.27)) hide)
+    )
