File: manufacturing/Reader_Module/MCU.kicad_sch (KiCad schematic)
At the start: 6 parts, among them J1 SW-Debug, U1 STM32L431KBU6

Commit message: added Matching NW to Schematic
Connections:
- net TRF_MOD is gone; now on net TRF_IRQ: U1.18 (PA8)
- net TRF_SYS_CLK is gone; now on net TRF_EN: U1.6 (PA0)
- net TRF_EN: no longer U1.3 (PC15)
- net TRF_IRQ: no longer U1.19 (PA9)
- net TRF_ASK_OOK: no longer names the net of U1.20 (PA10)
- no-connect marks 7 -> 10

Commit message: upd board
Parts:
- C4: LCSC Part # C1525 -> C2997286
- U1: LCSC Part # (none) -> C2826408
Changed lines of the file:
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@@
       (effects (font (size 1.27 1.27)) hide)
     )
-    (property "LCSC Part #" "C1525" (at 110.49 63.5 0)
+    (property "LCSC Part #" "C2997286" (at 110.49 63.5 0)
       (effects (font (size 1.27 1.27)) hide)
     )
@@
       (effects (font (size 1.27 1.27)) hide)
     )
+    (property "LCSC Part #" "C2826408" (at 168.91 111.76 0)
+      (effects (font (size 1.27 1.27)) hide)
+    )
