File: manufacturing/Reader_Module/RF.kicad_sch (KiCad schematic)
At the start: 0 parts

Commit message: added Matching NW to Schematic
Parts:
- added C30, C31: 1n5, Capacitor_SMD:C_0402_1005Metric, symbol Device:C
- added C32, C33: 1n2, Capacitor_SMD:C_0402_1005Metric, symbol Device:C
- added C34, C36: 680p, Capacitor_SMD:C_0402_1005Metric, symbol Device:C
- added C35: 220p, Capacitor_SMD:C_0402_1005Metric, symbol Device:C
- added C37: 100p, Capacitor_SMD:C_0402_1005Metric, symbol Device:C
- added C38: 47p, Capacitor_SMD:C_0402_1005Metric, symbol Device:C
- added L1, L2: 150n, Inductor_SMD:L_0805_2012Metric, symbol Device:L
- added R11: 0R, Resistor_SMD:R_0402_1005Metric, symbol Device:R
Connections:
- net RF_RX_IN1: now also C32.1, C33.2
- net RF_RX_IN2: now also C35.1, C36.2
- net RF_TX_OUT: now also C30.1, C31.2
- net SE_OUT: now also R11.2
- new net: C32.2, C34.2, L1.2, L2.1
- new net: C35.2, C37.2, C38.2, L2.2, R11.1
- new net: C30.2, C31.1, L1.1
- new net GND: C33.1, C34.1, C36.1, C37.1, C38.1
Other:
- note added: "4R to 50R"
- note added: "Phase Adj."
- note added: "VSWR Adj."

Commit message: upd board
Parts:
- C30: value 1n5 -> 1n2; LCSC Part # (none) -> C192386
- C31: value 1n5 -> 1n8; LCSC Part # (none) -> C527007
- C32, C33: LCSC Part # (none) -> C192386
- C34, C36: LCSC Part # (none) -> C1541
- C35: LCSC Part # (none) -> C1530
- C37: LCSC Part # (none) -> C1546
- C38: LCSC Part # (none) -> C1567
- L1, L2: LCSC Part # (none) -> C30618
Changed lines of the file:
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@@
+      (effects (font (size 1.27 1.27)) hide)
+    )
+    (property "LCSC Part #" "C192386" (at 93.98 115.57 0)
       (effects (font (size 1.27 1.27)) hide)
     )
@@
       (effects (font (size 1.27 1.27)) hide)
     )
+    (property "LCSC Part #" "C1541" (at 124.46 125.73 0)
+      (effects (font (size 1.27 1.27)) hide)
+    )
     (pin "1")
     (pin "2")
@@
       (effects (font (size 1.27 1.27)))
     )
-    (property "Value" "1n5" (at 81.28 109.22 90)
+    (property "Value" "1n2" (at 81.28 109.22 90)
       (effects (font (size 1.27 1.27)))
     )
@@
     )
     (property "Datasheet" "~" (at 77.47 110.49 0)
+      (effects (font (size 1.27 1.27)) hide)
+    )
+    (property "LCSC Part #" "C192386" (at 77.47 110.49 0)
       (effects (font (size 1.27 1.27)) hide)
     )
@@
       (effects (font (size 1.27 1.27)) hide)
     )
+    (property "LCSC Part #" "C30618" (at 88.9 110.49 0)
+      (effects (font (size 1.27 1.27)) hide)
+    )
     (pin "1")
     (pin "2")
@@
       (effects (font (size 1.27 1.27)) hide)
     )
+    (property "LCSC Part #" "C1541" (at 109.22 125.73 0)
+      (effects (font (size 1.27 1.27)) hide)
+    )
     (pin "1")
     (pin "2")
@@
       (effects (font (size 1.27 1.27)) hide)
     )
+    (property "LCSC Part #" "C1567" (at 146.05 115.57 0)
+      (effects (font (size 1.27 1.27)) hide)
+    )
     (pin "1")
     (pin "2")
@@
       (effects (font (size 1.27 1.27)) hide)
     )
+    (property "LCSC Part #" "C1546" (at 135.89 115.57 0)
+      (effects (font (size 1.27 1.27)) hide)
+    )
     (pin "1")
     (pin "2")
@@
       (effects (font (size 1.27 1.27)) hide)
     )
+    (property "LCSC Part #" "C1530" (at 124.46 115.57 0)
+      (effects (font (size 1.27 1.27)) hide)
+    )
     (pin "1")
     (pin "2")
@@
       (effects (font (size 1.27 1.27)))
     )
-    (property "Value" "1n5" (at 81.28 115.57 90)
+    (property "Value" "1n8" (at 81.28 115.57 90)
       (effects (font (size 1.27 1.27)))
     )
@@
       (effects (font (size 1.27 1.27)) hide)
     )
+    (property "LCSC Part #" "C527007" (at 77.47 116.84 0)
+      (effects (font (size 1.27 1.27)) hide)
+    )
     (pin "1")
     (pin "2")
@@
     )
     (property "Datasheet" "~" (at 93.98 125.73 0)
+      (effects (font (size 1.27 1.27)) hide)
+    )
+    (property "LCSC Part #" "C192386" (at 93.98 125.73 0)
       (effects (font (size 1.27 1.27)) hide)
     )
@@
       (effects (font (size 1.27 1.27)) hide)
     )
+    (property "LCSC Part #" "C30618" (at 116.84 110.49 0)
+      (effects (font (size 1.27 1.27)) hide)
+    )
