File: manufacturing/Reader_Module/Reader_Module.kicad_sch (KiCad schematic)
At the start: 7 parts

Commit message: added Matching NW to Schematic
Parts:
- removed H2: MountingHole_Pad, MountingHole:MountingHole_3.2mm_M3_Pad_Via, symbol Mechanical:MountingHole_Pad
- H3, H4: footprint MountingHole:MountingHole_3.2mm_M3_Pad_Via -> MountingHole:MountingHole_3.2mm_M3
Other:
- sheet MCU ports: added none; removed TRF_ASK_OOK, TRF_MOD, TRF_SYS_CLK
- sheet TRF ports: added none; removed TRF_ASK_OOK, TRF_MOD, TRF_SYS_CLK
- note added: "Mounting/Tooling"
- moved on the sheet: H1, H3, H4, H5, H6, H7

Commit message: upd board
Parts:
- removed H1: MountingHole_Pad, MountingHole:MountingHole_3.2mm_M3_Pad_Via, symbol Mechanical:MountingHole_Pad
- removed H3, H4: MountingHole_Pad, MountingHole:MountingHole_3.2mm_M3, symbol Mechanical:MountingHole_Pad
- removed H5, H6, H7: ~, JLC:JLC_Tooling, symbol JLC:Tooling_Hole
Other:
- note removed: "Mounting/Tooling"
Changed lines of the file:
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@@
-    (fill (type none))
-  )
-  (rectangle (start 139.7 88.9) (end 160.02 114.3)
-    (stroke (width 0) (type dash))
     (fill (type none))
   )
@@
     (effects (font (size 5.08 5.08) (thickness 1.016) bold italic) (justify left bottom))
   )
-  (text "Mounting/Tooling" (at 139.7 87.63 0)
-    (effects (font (size 1.27 1.27)) (justify left bottom))
-  )
   (text "RF" (at 100.33 85.09 0)
     (effects (font (size 2.54 2.54) bold) (justify right bottom))
@@
     (effects (font (size 2.54 2.54) bold) (justify left bottom))
   )
-  (symbol (lib_id "Mechanical:MountingHole_Pad") (at 144.78 102.87 0) (unit 1)
-    (in_bom yes) (on_board yes) (dnp no)
-    (property "Reference" "H4" (at 144.78 99.06 0)
-      (effects (font (size 1.27 1.27)) (justify bottom))
-    )
-    (property "Value" "MountingHole_Pad" (at 147.32 102.87 0)
-      (effects (font (size 1.27 1.27)) (justify left) hide)
-    )
-    (property "Footprint" "MountingHole:MountingHole_3.2mm_M3" (at 144.78 102.87 0)
-      (effects (font (size 1.27 1.27)) hide)
-    )
-    (property "Datasheet" "~" (at 144.78 102.87 0)
-      (effects (font (size 1.27 1.27)) hide)
-    )
-    (pin "1")
-    (instances
-      (project "Reader_Module"
-        (path "/a12f3265-d34f-4fd6-8a74-fc2a0f1ff00e"
-          (reference "H4") (unit 1)
-        )
-      )
-    )
-  )
-  (symbol (lib_id "Mechanical:MountingHole_Pad") (at 149.86 102.87 0) (unit 1)
-    (in_bom yes) (on_board yes) (dnp no)
-    (property "Reference" "H3" (at 149.86 99.06 0)
-      (effects (font (size 1.27 1.27)) (justify bottom))
-    )
-    (property "Value" "MountingHole_Pad" (at 152.4 102.87 0)
-      (effects (font (size 1.27 1.27)) (justify left) hide)
-    )
-    (property "Footprint" "MountingHole:MountingHole_3.2mm_M3" (at 149.86 102.87 0)
-      (effects (font (size 1.27 1.27)) hide)
-    )
-    (property "Datasheet" "~" (at 149.86 102.87 0)
-      (effects (font (size 1.27 1.27)) hide)
-    )
-    (pin "1")
-    (instances
-      (project "Reader_Module"
-        (path "/a12f3265-d34f-4fd6-8a74-fc2a0f1ff00e"
-          (reference "H3") (unit 1)
-        )
-      )
-    )
-  )
-  (symbol (lib_id "power:GND") (at 149.86 105.41 0) (unit 1)
-    (in_bom yes) (on_board yes) (dnp no)
-    (property "Reference" "#PWR033" (at 149.86 111.76 0)
-      (effects (font (size 1.27 1.27)) hide)
-    )
-    (property "Value" "GND" (at 149.86 109.22 0)
-      (effects (font (size 1.27 1.27)))
-    )
-    (property "Footprint" "" (at 149.86 105.41 0)
-      (effects (font (size 1.27 1.27)) hide)
-    )
-    (property "Datasheet" "" (at 149.86 105.41 0)
-      (effects (font (size 1.27 1.27)) hide)
-    )
-    (pin "1")
-    (instances
-      (project "STM32F4_HexGauge_V3"
-        (path "/1671c3d2-535f-4cd5-a65b-02e5c9ad18e5/2ad56a2f-dfcc-4b7b-a763-7659f3fc7ffe"
-          (reference "#PWR033") (unit 1)
-        )
-      )
-      (project "Reader_Module"
-        (path "/a12f3265-d34f-4fd6-8a74-fc2a0f1ff00e/74619374-293a-4fe1-b841-17e202b00b2f"
-          (reference "#PWR031") (unit 1)
-        )
-        (path "/a12f3265-d34f-4fd6-8a74-fc2a0f1ff00e"
-          (reference "#PWR035") (unit 1)
-        )
-      )
-    )
-  )
-  (symbol (lib_id "JLC:Tooling_Hole") (at 154.94 95.25 0) (unit 1)
-    (in_bom yes) (on_board yes) (dnp no)
-    (property "Reference" "H7" (at 153.67 92.71 0)
-      (effects (font (size 1.27 1.27)) (justify left))
-    )
-    (property "Value" "~" (at 153.67 95.25 0)
-      (effects (font (size 1.27 1.27)))
-    )
-    (property "Footprint" "JLC:JLC_Tooling" (at 153.67 100.33 0)
-      (effects (font (size 1.27 1.27)) hide)
-    )
-    (property "Datasheet" "https://jlcpcb.com/help/article/47-How-to-add-tooling-holes-for-PCB-assembly-order" (at 153.67 97.79 0)
-      (effects (font (size 1.27 1.27)) hide)
-    )
-    (instances
-      (project "Reader_Module"
-        (path "/a12f3265-d34f-4fd6-8a74-fc2a0f1ff00e"
-          (reference "H7") (unit 1)
-        )
-      )
-    )
-  )
-  (symbol (lib_id "JLC:Tooling_Hole") (at 149.86 95.25 0) (unit 1)
-    (in_bom yes) (on_board yes) (dnp no)
-    (property "Reference" "H6" (at 148.59 92.71 0)
-      (effects (font (size 1.27 1.27)) (justify left))
-    )
-    (property "Value" "~" (at 148.59 95.25 0)
-      (effects (font (size 1.27 1.27)))
-    )
-    (property "Footprint" "JLC:JLC_Tooling" (at 148.59 100.33 0)
-      (effects (font (size 1.27 1.27)) hide)
-    )
-    (property "Datasheet" "https://jlcpcb.com/help/article/47-How-to-add-tooling-holes-for-PCB-assembly-order" (at 148.59 97.79 0)
-      (effects (font (size 1.27 1.27)) hide)
-    )
-    (instances
-      (project "Reader_Module"
-        (path "/a12f3265-d34f-4fd6-8a74-fc2a0f1ff00e"
-          (reference "H6") (unit 1)
-        )
-      )
-    )
-  )
-  (symbol (lib_id "JLC:Tooling_Hole") (at 144.78 95.25 0) (unit 1)
-    (in_bom yes) (on_board yes) (dnp no)
-    (property "Reference" "H5" (at 143.51 92.71 0)
-      (effects (font (size 1.27 1.27)) (justify left))
-    )
-    (property "Value" "~" (at 143.51 95.25 0)
-      (effects (font (size 1.27 1.27)))
-    )
-    (property "Footprint" "JLC:JLC_Tooling" (at 143.51 100.33 0)
-      (effects (font (size 1.27 1.27)) hide)
-    )
-    (property "Datasheet" "https://jlcpcb.com/help/article/47-How-to-add-tooling-holes-for-PCB-assembly-order" (at 143.51 97.79 0)
-      (effects (font (size 1.27 1.27)) hide)
-    )
-    (instances
-      (project "Reader_Module"
-        (path "/a12f3265-d34f-4fd6-8a74-fc2a0f1ff00e"
-          (reference "H5") (unit 1)
-        )
-      )
-    )
-  )
-  (symbol (lib_id "Mechanical:MountingHole_Pad") (at 154.94 102.87 0) (unit 1)
-    (in_bom yes) (on_board yes) (dnp no)
-    (property "Reference" "H1" (at 154.94 99.06 0)
-      (effects (font (size 1.27 1.27)) (justify bottom))
-    )
-    (property "Value" "MountingHole_Pad" (at 157.48 102.87 0)
-      (effects (font (size 1.27 1.27)) (justify left) hide)
-    )
-    (property "Footprint" "MountingHole:MountingHole_3.2mm_M3_Pad_Via" (at 154.94 102.87 0)
-      (effects (font (size 1.27 1.27)) hide)
-    )
-    (property "Datasheet" "~" (at 154.94 102.87 0)
-      (effects (font (size 1.27 1.27)) hide)
-    )
-    (pin "1")
-    (instances
-      (project "Reader_Module"
-        (path "/a12f3265-d34f-4fd6-8a74-fc2a0f1ff00e"
-          (reference "H1") (unit 1)
-        )
-      )
-    )
-  )
-  (symbol (lib_id "power:GND") (at 154.94 105.41 0) (unit 1)
-    (in_bom yes) (on_board yes) (dnp no)
-    (property "Reference" "#PWR033" (at 154.94 111.76 0)
-      (effects (font (size 1.27 1.27)) hide)
-    )
-    (property "Value" "GND" (at 154.94 109.22 0)
-      (effects (font (size 1.27 1.27)))
-    )
-    (property "Footprint" "" (at 154.94 105.41 0)
-      (effects (font (size 1.27 1.27)) hide)
-    )
-    (property "Datasheet" "" (at 154.94 105.41 0)
-      (effects (font (size 1.27 1.27)) hide)
-    )
-    (pin "1")
-    (instances
-      (project "STM32F4_HexGauge_V3"
-        (path "/1671c3d2-535f-4cd5-a65b-02e5c9ad18e5/2ad56a2f-dfcc-4b7b-a763-7659f3fc7ffe"
-          (reference "#PWR033") (unit 1)
-        )
-      )
-      (project "Reader_Module"
-        (path "/a12f3265-d34f-4fd6-8a74-fc2a0f1ff00e/74619374-293a-4fe1-b841-17e202b00b2f"
-          (reference "#PWR031") (unit 1)
-        )
-        (path "/a12f3265-d34f-4fd6-8a74-fc2a0f1ff00e"
-          (reference "#PWR037") (unit 1)
-        )
-      )
-    )
-  )
-  (symbol (lib_id "power:GND") (at 144.78 105.41 0) (unit 1)
-    (in_bom yes) (on_board yes) (dnp no)
-    (property "Reference" "#PWR033" (at 144.78 111.76 0)
-      (effects (font (size 1.27 1.27)) hide)
-    )
-    (property "Value" "GND" (at 144.78 109.22 0)
-      (effects (font (size 1.27 1.27)))
-    )
-    (property "Footprint" "" (at 144.78 105.41 0)
-      (effects (font (size 1.27 1.27)) hide)
-    )
-    (property "Datasheet" "" (at 144.78 105.41 0)
-      (effects (font (size 1.27 1.27)) hide)
-    )
-    (pin "1")
-    (instances
-      (project "STM32F4_HexGauge_V3"
-        (path "/1671c3d2-535f-4cd5-a65b-02e5c9ad18e5/2ad56a2f-dfcc-4b7b-a763-7659f3fc7ffe"
-          (reference "#PWR033") (unit 1)
-        )
-      )
-      (project "Reader_Module"
-        (path "/a12f3265-d34f-4fd6-8a74-fc2a0f1ff00e/74619374-293a-4fe1-b841-17e202b00b2f"
-          (reference "#PWR031") (unit 1)
-        )
-        (path "/a12f3265-d34f-4fd6-8a74-fc2a0f1ff00e"
-          (reference "#PWR024") (unit 1)
-        )
-      )
-    )
-  )
   (sheet (at 114.3 63.5) (size 25.4 12.7) (fields_autoplaced)
