File: manufacturing/Reader_Module/Strapping.kicad_sch (KiCad schematic)
At the start: 7 parts, among them SW1 NRST

Commit message: upd board
Parts:
- C7: value 1u -> 2u2; LCSC Part # (none) -> C2997286
- D2: LCSC Part # (none) -> C2296
- R1: LCSC Part # (none) -> C25792
- R2: LCSC Part # (none) -> C25744
- R4: value 1k -> 1k5; LCSC Part # (none) -> C25741
- SW1: LCSC Part # (none) -> C79174
Changed lines of the file:
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@@
+      (effects (font (size 1.27 1.27)) hide)
+    )
+    (property "LCSC Part #" "C25744" (at 187.96 95.25 0)
       (effects (font (size 1.27 1.27)) hide)
     )
@@
     )
     (property "Datasheet" "https://omronfs.omron.com/en_US/ecb/products/pdf/en-b3fs.pdf" (at 102.87 88.9 0)
+      (effects (font (size 1.27 1.27)) hide)
+    )
+    (property "LCSC Part #" "C79174" (at 102.87 93.98 0)
       (effects (font (size 1.27 1.27)) hide)
     )
@@
       (effects (font (size 1.27 1.27)) hide)
     )
+    (property "LCSC Part #" "C25792" (at 109.22 88.9 0)
+      (effects (font (size 1.27 1.27)) hide)
+    )
     (pin "1")
     (pin "2")
@@
       (effects (font (size 1.27 1.27)) hide)
     )
+    (property "LCSC Part #" "C2296" (at 148.59 90.17 0)
+      (effects (font (size 1.27 1.27)) hide)
+    )
     (pin "1")
     (pin "2")
@@
       (effects (font (size 1.27 1.27)) (justify top))
     )
-    (property "Value" "1u" (at 105.41 100.33 90)
+    (property "Value" "2u2" (at 106.68 100.33 90)
       (effects (font (size 1.27 1.27)) (justify top))
     )
@@
       (effects (font (size 1.27 1.27)) hide)
     )
+    (property "LCSC Part #" "C2997286" (at 102.87 101.6 0)
+      (effects (font (size 1.27 1.27)) hide)
+    )
     (pin "1")
     (pin "2")
@@
       (effects (font (size 1.27 1.27)) (justify left))
     )
-    (property "Value" "1k" (at 149.86 101.6 0)
+    (property "Value" "1k5" (at 149.86 101.6 0)
       (effects (font (size 1.27 1.27)) (justify left))
     )
@@
       (effects (font (size 1.27 1.27)) hide)
     )
+    (property "LCSC Part #" "C25741" (at 148.59 100.33 0)
+      (effects (font (size 1.27 1.27)) hide)
+    )
