File: manufacturing/Reader_Module/TRF.kicad_sch (KiCad schematic)
At the start: 15 parts, among them Y1 13.56MHz

Commit message: added Matching NW to Schematic
Connections:
- net TRF_ASK_OOK: no longer names the net of D1.12 (ASK/OOK)
- net TRF_SYS_CLK: no longer names the net of D1.27 (SYS_CLK)
- no-connect marks 0 -> 2
Other:
- note added: "direct mode only"
- note added: "use HSI RC"
Changed lines of the file:
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@@
 (kicad_sch (version 20230121) (generator eeschema)
   (paper "A4")
+  (title_block
+    (date "2023-08-15")
+    (rev "R0")
+  )
   (junction (at 200.66 58.42) (diameter 0) (color 0 0 0 0)
   )
@@
   (junction (at 92.71 49.53) (diameter 0) (color 0 0 0 0)
   )
+  (no_connect (at 45.72 69.85))
+  (no_connect (at 45.72 97.79))
   (wire (pts (xy 43.18 77.47) (xy 45.72 77.47))
     (stroke (width 0) (type default))
@@
     (stroke (width 0) (type default))
   )
-  (wire (pts (xy 43.18 97.79) (xy 45.72 97.79))
-    (stroke (width 0) (type default))
-  )
   (wire (pts (xy 92.71 87.63) (xy 91.44 87.63))
     (stroke (width 0) (type default))
@@
   )
   (wire (pts (xy 162.56 68.58) (xy 162.56 67.31))
-    (stroke (width 0) (type default))
-  )
-  (wire (pts (xy 43.18 69.85) (xy 45.72 69.85))
     (stroke (width 0) (type default))
   )
@@
     (fill (type none))
   )
-  (text_box "NOTES:\nVDD_X as 3V3 Power output for MCU\n"
+  (text_box "NOTES:\nVDD_X as 3V3 Power output for MCU\nParallel (non direct) interface"
     (at 25.4 165.1 0) (size 139.7 25.4)
     (stroke (width 0) (type default))
@@
     (effects (font (size 1.27 1.27)) (justify left top))
   )
+  (text "use HSI RC" (at 44.45 71.12 0)
+    (effects (font (size 1.27 1.27)) (justify right bottom) (href "#2"))
+  )
+  (text "direct mode only" (at 44.45 99.06 0)
+    (effects (font (size 1.27 1.27)) (justify right bottom))
+  )
   (text "Decoupling" (at 114.3 49.53 0)
     (effects (font (size 1.27 1.27)) (justify left bottom))
@@
     (effects (font (size 1.27 1.27)) (justify right))
   )
-  (hierarchical_label "TRF_ASK_OOK" (shape bidirectional) (at 43.18 97.79 180) (fields_autoplaced)
-    (effects (font (size 1.27 1.27)) (justify right))
-  )
   (hierarchical_label "RF_TX_OUT" (shape output) (at 92.71 80.01 0) (fields_autoplaced)
     (effects (font (size 1.27 1.27)) (justify left))
@@
     (effects (font (size 1.27 1.27) italic) (justify right))
   )
-  (hierarchical_label "TRF_SYS_CLK" (shape output) (at 43.18 69.85 180) (fields_autoplaced)
-    (effects (font (size 1.27 1.27)) (justify right))
-  )
   (hierarchical_label "TRF_IO_5" (shape bidirectional) (at 43.18 87.63 180) (fields_autoplaced)

Commit message: upd board
Parts:
- C10, C12, C14, C16, C18: LCSC Part # (none) -> C15195
- C11, C13, C15, C17, C9: LCSC Part # C1525 -> C2997286
- C5, C6: value 27pF -> 27p; LCSC Part # (none) -> C1557
- D1: LCSC Part # (none) -> C2654840
- R3: LCSC Part # (none) -> C25076
- Y1: LCSC Part # (none) -> C164051
Changed lines of the file:
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@@
+      (effects (font (size 1.27 1.27)) hide)
+    )
+    (property "LCSC Part #" "C15195" (at 190.5 63.5 0)
       (effects (font (size 1.27 1.27)) hide)
     )
@@
     (property "Arrow Price/Stock" "https://www.arrow.com/en/products/trf7964arhbr/texas-instruments" (at 82.55 1039.37 0)
       (effects (font (size 1.27 1.27)) (justify left top) hide)
+    )
+    (property "LCSC Part #" "C2654840" (at 50.8 57.15 0)
+      (effects (font (size 1.27 1.27)) hide)
     )
     (pin "1")
@@
       (effects (font (size 1.27 1.27)) hide)
     )
-    (property "LCSC Part #" "C1525" (at 143.51 63.5 0)
+    (property "LCSC Part #" "C2997286" (at 143.51 63.5 0)
       (effects (font (size 1.27 1.27)) hide)
     )
@@
       (effects (font (size 1.27 1.27)) (justify right))
     )
-    (property "Value" "27pF" (at 139.7 100.33 0)
+    (property "Value" "27p" (at 139.7 100.33 0)
       (effects (font (size 1.27 1.27)) (justify right))
     )
@@
       (effects (font (size 1.27 1.27)) hide)
     )
+    (property "LCSC Part #" "C1557" (at 142.24 99.06 0)
+      (effects (font (size 1.27 1.27)) hide)
+    )
     (pin "1")
     (pin "2")
@@
       (effects (font (size 1.27 1.27)) (justify right))
     )
-    (property "Value" "27pF" (at 121.92 100.33 0)
+    (property "Value" "27p" (at 121.92 100.33 0)
       (effects (font (size 1.27 1.27)) (justify right))
     )
@@
     )
     (property "Datasheet" "~" (at 124.46 99.06 0)
+      (effects (font (size 1.27 1.27)) hide)
+    )
+    (property "LCSC Part #" "C1557" (at 124.46 99.06 0)
       (effects (font (size 1.27 1.27)) hide)
     )
@@
       (effects (font (size 1.27 1.27)) hide)
     )
-    (property "LCSC Part #" "C1525" (at 162.56 63.5 0)
+    (property "LCSC Part #" "C2997286" (at 162.56 63.5 0)
       (effects (font (size 1.27 1.27)) hide)
     )
@@
     )
     (property "Datasheet" "~" (at 209.55 63.5 0)
+      (effects (font (size 1.27 1.27)) hide)
+    )
+    (property "LCSC Part #" "C15195" (at 209.55 63.5 0)
       (effects (font (size 1.27 1.27)) hide)
     )
@@
       (effects (font (size 1.27 1.27)) hide)
     )
+    (property "LCSC Part #" "C164051" (at 133.35 93.98 0)
+      (effects (font (size 1.27 1.27)) hide)
+    )
     (pin "1")
     (pin "2")
@@
       (effects (font (size 1.27 1.27)) hide)
     )
+    (property "LCSC Part #" "C15195" (at 152.4 63.5 0)
+      (effects (font (size 1.27 1.27)) hide)
+    )
     (pin "1")
     (pin "2")
@@
       (effects (font (size 1.27 1.27)) hide)
     )
-    (property "LCSC Part #" "C1525" (at 181.61 63.5 0)
+    (property "LCSC Part #" "C2997286" (at 181.61 63.5 0)
       (effects (font (size 1.27 1.27)) hide)
     )
@@
       (effects (font (size 1.27 1.27)) hide)
     )
+    (property "LCSC Part #" "C15195" (at 171.45 63.5 0)
+      (effects (font (size 1.27 1.27)) hide)
+    )
     (pin "1")
     (pin "2")
@@
       (effects (font (size 1.27 1.27)) hide)
     )
-    (property "LCSC Part #" "C1525" (at 124.46 63.5 0)
+    (property "LCSC Part #" "C2997286" (at 124.46 63.5 0)
       (effects (font (size 1.27 1.27)) hide)
     )
@@
       (effects (font (size 1.27 1.27)) hide)
     )
+    (property "LCSC Part #" "C25076" (at 92.71 54.61 0)
+      (effects (font (size 1.27 1.27)) hide)
+    )
     (pin "1")
     (pin "2")
@@
       (effects (font (size 1.27 1.27)) hide)
     )
+    (property "LCSC Part #" "C15195" (at 133.35 63.5 0)
+      (effects (font (size 1.27 1.27)) hide)
+    )
     (pin "1")
     (pin "2")
@@
       (effects (font (size 1.27 1.27)) hide)
     )
-    (property "LCSC Part #" "C1525" (at 200.66 63.5 0)
-      (effects (font (size 1.27 1.27)) hide)
-    )
+    (property "LCSC Part #" "C2997286" (at 200.66 63.5 0)
+      (effects (font (size 1.27 1.27)) hide)
+    )
